Commit message: makes top of velodyne invisble to camera

File: catkin_ws/src/bowser_sim/models/bowser2/model.urdf (robot description, URDF)
Before this commit: robot bowser2, 6 links, 5 joints
Links:
- link bowser2/bowser_hdl32/hdl32_top: geometry collision cylinder length=0.07357 radius=0.04267

Commit message: first attempts at navigation stack

File: catkin_ws/src/bowser_sim/models/bowser2/model.urdf (robot description, URDF)
Before this commit: robot bowser2, 6 links, 5 joints
Links:
- link bowser2/bowser_hdl32/hdl32_top: geometry collision cylinder length=0.07357 radius=0.04267; visual mesh filename=package://bowser_sim/models/bowser_hdl32/meshes/velodyne_to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 scale=1.0 1.0 1.0
Joints:
- joint bowser2/depthcam_joint: origin xyz=0     0     0.9548 rpy=1.5708      3.14159      -1.5708 -> xyz=-0.35  0    0.7 rpy=0      0      3.14159
- joint bowser2/hdl32_joint: origin xyz=-0.35     0       0.72933 rpy=0      0      3.14159 -> xyz=0      0      1.22933 rpy=0      0      3.14159

Commit message: implements working mapping with depth cam

File: catkin_ws/src/bowser_sim/models/bowser2/model.urdf (robot description, URDF)
Before this commit: robot bowser2, 6 links, 5 joints
Joints:
- joint bowser2/depthcam_joint: origin xyz=-0.35  0    0.7 rpy=0      0      3.14159 -> xyz=-0.35   0     0.236 rpy=-1.5708   0       1.57079
- joint bowser2/front_left_joint: origin xyz=-0.3  -0.37  0.45 rpy=0 0 0 -> xyz=-0.3  -0.37 -0.05 rpy=0 0 0
- joint bowser2/front_right_joint: origin xyz=-0.3   0.37  0.45 rpy=0 0 0 -> xyz=-0.3   0.37 -0.05 rpy=0 0 0
- joint bowser2/hdl32_joint: origin xyz=0      0      1.22933 rpy=0      0      3.14159 -> xyz=0      0      0.42933 rpy=0      0      3.14159
